Commit message: fix WRT problem

File: ros_pack/urdf_tutorial_r2d2/urdf/4arms.urdf (robot description, URDF)
Before this commit: robot 4ArmDrone, 9 links, 8 joints
Joints:
- joint base_to_arm_1: origin xyz=${xd+0.029} ${yd} 0 rpy=0 0 2.15 -> xyz=-0.07100000000000001 0.05 0 rpy=0 0 2.15
- joint base_to_arm_2: origin xyz=${xd+0.029} ${yd-0.093} 0 rpy=0 0 -2.15 -> xyz=-0.07100000000000001 -0.043 0 rpy=0 0 -2.15
- joint base_to_arm_3: origin xyz=${xd+0.165} ${yd-0.093} 0 rpy=0 0 -1 -> xyz=0.065 -0.043 0 rpy=0 0 -1
- joint base_to_arm_4: origin xyz=${xd+0.165} ${yd} 0 rpy=0 0 1 -> xyz=0.065 0.05 0 rpy=0 0 1

Commit message: correct torque at X, but Y still wrong

File: ros_pack/urdf_tutorial_r2d2/urdf/4arms.urdf (robot description, URDF)
Before this commit: robot 4ArmDrone, 9 links, 8 joints
Joints:
- joint base_to_arm_1: origin xyz=-0.07100000000000001 0.05 0 rpy=0 0 2.15 -> xyz=-0.06906999999999999 0.046645 0 rpy=0 0 2.1495963267948968
- joint base_to_arm_2: origin xyz=-0.07100000000000001 -0.043 0 rpy=0 0 -2.15 -> xyz=-0.06906999999999999 -0.046355 0 rpy=0 0 -2.1495963267948968
- joint base_to_arm_3: origin xyz=0.065 -0.043 0 rpy=0 0 -1 -> xyz=0.06906999999999999 -0.046355 0 rpy=0 0 -0.9919963267948966
- joint base_to_arm_4: origin xyz=0.065 0.05 0 rpy=0 0 1 -> xyz=0.06906999999999999 0.046645 0 rpy=0 0 0.9919963267948966
- joint prop_to_arm_1: origin xyz=0.17 0.02 0.03 rpy=0 0 0 -> xyz=0.155 0.0175 0.035 rpy=0 0 0
- joint prop_to_arm_2: axis 0.0 0.0 -1 -> 0.0 0.0 1; origin xyz=0.17 -0.02 0.03 rpy=0 0 0 -> xyz=0.155 -0.0175 0.035 rpy=0 0 0
- joint prop_to_arm_3: origin xyz=0.17 0.02 0.03 rpy=0 0 0 -> xyz=0.155 0.0175 0.035 rpy=0 0 0
- joint prop_to_arm_4: axis 0.0 0.0 -1 -> 0.0 0.0 1; origin xyz=0.17 -0.02 0.03 rpy=0 0 0 -> xyz=0.155 -0.0175 0.035 rpy=0 0 0

File: ros_pack/urdf_tutorial_r2d2/urdf/4arms.urdf.xacro (robot description, xacro)
@@ -1,9 +1,15 @@
 <?xml version="1.0"?>
-<robot name="4ArmDrone"  xmlns:xacro="http://www.ros.org/wiki/xacro">
+<robot name="4Armdrone"  xmlns:xacro="http://www.ros.org/wiki/xacro">
   <material name="blue">
     <color rgba="0 0 0.8 1"/>
   </material>
-<xacro:property name="xd" value="-0.1"/>
-<xacro:property name="yd" value="0.05"/>
+<xacro:property name='sktX' value="0.19674"/>
+<xacro:property name='sktY' value="0.09329"/>
+<xacro:property name="xd"   value="${-sktX/2}"/>
+<xacro:property name="yd"   value="${sktY/2}"/>
+<xacro:property name="arm_junction" value="0.0293"/>
+<xacro:property name="arm_base" value="0.035"/>
+<xacro:property name="arm_ang" value="0.5788"/>
+<xacro:property name="arm_len" value="0.155"/>
   <link name="drone">
     <visual name="drone_visual">
@@ -29,4 +35,5 @@
               scale="0.001 0.001 0.001"/>
       </geometry>
+      <origin xyz="0 ${0} 0"/>
     </visual>
     <collision>
@@ -35,4 +42,5 @@
               scale="0.001 0.001 0.001"/>
       </geometry>
+      <origin xyz="0 ${0} 0"/>
     </collision>
   </link>
@@ -43,8 +51,8 @@
             scale="0.001 0.001 0.001"/>
       </geometry>
-      <origin xyz="0 -0.035 0"/>
+      <origin xyz="0 ${-arm_base} 0"/>
     </visual>
     <collision>
-      <origin xyz="0 -0.035 0"/>
+      <origin xyz="0 ${-arm_base} 0"/>
       <geometry>
         <mesh filename="package://urdf_tutorial/meshes/Gazebo_Base_arm.STL"
@@ -59,4 +67,5 @@
               scale="0.001 0.001 0.001"/>
       </geometry>
+      <origin xyz="0 ${0} 0"/>
     </visual>
     <collision>
@@ -65,4 +74,5 @@
               scale="0.001 0.001 0.001"/>
       </geometry>
+      <origin xyz="0 ${0} 0"/>
     </collision>
   </link>
@@ -73,5 +83,5 @@
               scale="0.001 0.001 0.001"/>
       </geometry>
-      <origin xyz="0 -0.035 0"/>
+      <origin xyz="0 ${-arm_base} 0"/>
     </visual>
     <collision>
@@ -80,5 +90,5 @@
               scale="0.001 0.001 0.001"/>
       </geometry>
-      <origin xyz="0 -0.035 0"/>
+      <origin xyz="0 ${-arm_base} 0"/>
     </collision>
   </link>
@@ -86,5 +96,5 @@
     <parent link="drone"/>
     <child link="arm_1"/>
-    <origin  rpy="0 0 2.15" xyz="${xd+0.029} ${yd} 0"/>
+    <origin  rpy="0 0 ${pi/2+arm_ang}" xyz="${xd+arm_junction} ${yd} 0"/>
     <axis xyz="0.0 1.0 0.0"/>
     <limit effort="1000.0" lower="0.0" upper="1.74" velocity="1000.0"/>
@@ -93,5 +103,5 @@
     <parent link="drone"/>
     <child link="arm_2"/>
-    <origin  rpy="0 0 -2.15" xyz="${xd+0.029} ${yd-0.093} 0"/>
+    <origin  rpy="0 0 -${pi/2+arm_ang}" xyz="${xd+arm_junction} ${yd-0.093} 0"/>
     <axis xyz="0.0 1.0 0.0"/>
     <limit effort="1000.0" lower="0.0" upper="1.74" velocity="1000.0"/>
@@ -100,5 +110,5 @@
     <parent link="drone"/>
     <child link="arm_3"/>
-    <origin  rpy="0 0 -1" xyz="${xd+0.165} ${yd-0.093} 0"/>
+    <origin  rpy="0 0 -${pi/2-arm_ang}" xyz="${-xd-arm_junction} ${yd-0.093} 0"/>
     <axis xyz="0.0 1.0 0.0"/>
     <limit effort="1000.0" lower="0.0" upper="1.74" velocity="1000.0"/>
@@ -107,5 +117,5 @@
     <parent link="drone"/>
     <child link="arm_4"/>
-    <origin  rpy="0 0 1" xyz="${xd+0.165} ${yd} 0"/>
+    <origin  rpy="0 0 ${pi/2-arm_ang}" xyz="${-xd-arm_junction} ${yd} 0"/>
     <axis xyz="0.0 1.0 0.0"/>
     <limit effort="1000.0" lower="0.0" upper="1.74" velocity="1000.0"/>
@@ -122,5 +132,5 @@
     <parent link="arm_1"/>
     <child link="prop_1"/>
-    <origin  rpy="0 0 0" xyz="0.17 0.02 0.03"/>
+    <origin  rpy="0 0 0" xyz="${arm_len} ${arm_base/2} ${arm_base}"/>
     <axis xyz="0.0 0.0 1"/>
   </joint>
@@ -136,6 +146,6 @@
     <parent link="arm_2"/>
     <child link="prop_2"/>
-    <origin  rpy="0 0 0" xyz="0.17 -0.02 0.03"/>
-    <axis xyz="0.0 0.0 -1"/>
+    <origin  rpy="0 0 0" xyz="${arm_len} ${-arm_base/2} ${arm_base}"/>
+    <axis xyz="0.0 0.0 1"/>
   </joint>
   <link name="prop_3">
@@ -150,5 +160,5 @@
     <parent link="arm_3"/>
     <child link="prop_3"/>
-    <origin  rpy="0 0 0" xyz="0.17 0.02 0.03"/>
+    <origin  rpy="0 0 0" xyz="${arm_len} ${arm_base/2} ${arm_base}"/>
     <axis xyz="0.0 0.0 1"/>
   </joint>
@@ -164,6 +174,6 @@
     <parent link="arm_4"/>
     <child link="prop_4"/>
-    <origin  rpy="0 0 0" xyz="0.17 -0.02 0.03"/>
-    <axis xyz="0.0 0.0 -1"/>
+    <origin  rpy="0 0 0" xyz="${arm_len} ${-arm_base/2} ${arm_base}"/>
+    <axis xyz="0.0 0.0 1"/>
   </joint>
 </robot>

Commit message: on a un simulateur

File: ros_pack/urdf_tutorial_r2d2/urdf/4arms.urdf (robot description, URDF)
Before this commit: robot 4Armdrone, 9 links, 8 joints
Joints:
- joint base_to_arm_2: origin xyz=-0.06906999999999999 -0.046355 0 rpy=0 0 -2.1495963267948968 -> xyz=-0.06906999999999999 -0.046645 0 rpy=0 0 -2.1495963267948968
- joint base_to_arm_3: origin xyz=0.06906999999999999 -0.046355 0 rpy=0 0 -0.9919963267948966 -> xyz=0.06906999999999999 -0.046645 0 rpy=0 0 -0.9919963267948966
- joint prop_to_arm_1: origin xyz=0.155 0.0175 0.035 rpy=0 0 0 -> xyz=0.155 0.0175 0 rpy=0 0 0
- joint prop_to_arm_2: origin xyz=0.155 -0.0175 0.035 rpy=0 0 0 -> xyz=0.155 -0.0175 0 rpy=0 0 0
- joint prop_to_arm_3: origin xyz=0.155 0.0175 0.035 rpy=0 0 0 -> xyz=0.155 0.0175 0 rpy=0 0 0
- joint prop_to_arm_4: origin xyz=0.155 -0.0175 0.035 rpy=0 0 0 -> xyz=0.155 -0.0175 0 rpy=0 0 0

File: ros_pack/urdf_tutorial_r2d2/urdf/4arms.urdf.xacro (robot description, xacro)
@@ -103,5 +103,5 @@
     <parent link="drone"/>
     <child link="arm_2"/>
-    <origin  rpy="0 0 -${pi/2+arm_ang}" xyz="${xd+arm_junction} ${yd-0.093} 0"/>
+    <origin  rpy="0 0 -${pi/2+arm_ang}" xyz="${xd+arm_junction} ${-yd} 0"/>
     <axis xyz="0.0 1.0 0.0"/>
     <limit effort="1000.0" lower="0.0" upper="1.74" velocity="1000.0"/>
@@ -110,5 +110,5 @@
     <parent link="drone"/>
     <child link="arm_3"/>
-    <origin  rpy="0 0 -${pi/2-arm_ang}" xyz="${-xd-arm_junction} ${yd-0.093} 0"/>
+    <origin  rpy="0 0 -${pi/2-arm_ang}" xyz="${-xd-arm_junction} ${-yd} 0"/>
     <axis xyz="0.0 1.0 0.0"/>
     <limit effort="1000.0" lower="0.0" upper="1.74" velocity="1000.0"/>
@@ -132,5 +132,5 @@
     <parent link="arm_1"/>
     <child link="prop_1"/>
-    <origin  rpy="0 0 0" xyz="${arm_len} ${arm_base/2} ${arm_base}"/>
+    <origin  rpy="0 0 0" xyz="${arm_len} ${arm_base/2} ${0}"/>
     <axis xyz="0.0 0.0 1"/>
   </joint>
@@ -146,5 +146,5 @@
     <parent link="arm_2"/>
     <child link="prop_2"/>
-    <origin  rpy="0 0 0" xyz="${arm_len} ${-arm_base/2} ${arm_base}"/>
+    <origin  rpy="0 0 0" xyz="${arm_len} ${-arm_base/2} ${0}"/>
     <axis xyz="0.0 0.0 1"/>
   </joint>
@@ -160,5 +160,5 @@
     <parent link="arm_3"/>
     <child link="prop_3"/>
-    <origin  rpy="0 0 0" xyz="${arm_len} ${arm_base/2} ${arm_base}"/>
+    <origin  rpy="0 0 0" xyz="${arm_len} ${arm_base/2} ${0}"/>
     <axis xyz="0.0 0.0 1"/>
   </joint>
@@ -174,5 +174,5 @@
     <parent link="arm_4"/>
     <child link="prop_4"/>
-    <origin  rpy="0 0 0" xyz="${arm_len} ${-arm_base/2} ${arm_base}"/>
+    <origin  rpy="0 0 0" xyz="${arm_len} ${-arm_base/2} ${0}"/>
     <axis xyz="0.0 0.0 1"/>
   </joint>

Commit message: almost working again

File: ros_pack/urdf_tutorial_r2d2/urdf/4arms.urdf (robot description, URDF)
Before this commit: robot 4Armdrone, 9 links, 8 joints
Links:
- link arm_1: geometry collision mesh filename=package://urdf_tutorial_r2d2/meshes/Gazebo_Base_arm.STL scale=0.001 0.001 0.001; visual mesh filename=package://urdf_tutorial_r2d2/meshes/Gazebo_Base_arm.STL scale=0.001 0.001 0.001
- link arm_2: geometry collision mesh filename=package://urdf_tutorial_r2d2/meshes/Gazebo_Base_arm.STL scale=0.001 0.001 0.001; visual mesh filename=package://urdf_tutorial_r2d2/meshes/Gazebo_Base_arm.STL scale=0.001 0.001 0.001
- link arm_3: geometry collision mesh filename=package://urdf_tutorial_r2d2/meshes/Gazebo_Base_arm.STL scale=0.001 0.001 0.001; visual mesh filename=package://urdf_tutorial_r2d2/meshes/Gazebo_Base_arm.STL scale=0.001 0.001 0.001
- link arm_4: geometry collision mesh filename=package://urdf_tutorial_r2d2/meshes/Gazebo_Base_arm.STL scale=0.001 0.001 0.001; visual mesh filename=package://urdf_tutorial_r2d2/meshes/Gazebo_Base_arm.STL scale=0.001 0.001 0.001
- link drone: geometry collision mesh filename=package://urdf_tutorial_r2d2/meshes/Gazebo_Base_Body.STL scale=0.001 0.001 0.001; visual mesh filename=package://urdf_tutorial_r2d2/meshes/Gazebo_Base_Body.STL scale=0.001 0.001 0.001
- link prop_1: geometry visual mesh filename=package://urdf_tutorial_r2d2/meshes/1345_prop_ccw.STL
- link prop_2: geometry visual mesh filename=package://urdf_tutorial_r2d2/meshes/1345_prop_cw.STL
- link prop_3: geometry visual mesh filename=package://urdf_tutorial_r2d2/meshes/1345_prop_ccw.STL
- link prop_4: geometry visual mesh filename=package://urdf_tutorial_r2d2/meshes/1345_prop_cw.STL

File: ros_pack/urdf_tutorial_r2d2/urdf/4arms.urdf.xacro (robot description, xacro)
@@ -16,5 +16,5 @@
       <origin xyz="${xd} ${yd} 0" rpy="1.57079 0 0"/>
       <geometry>
-        <mesh filename="package://urdf_tutorial/meshes/Gazebo_Base_Body.STL"
+        <mesh filename="package://urdf_tutorial_r2d2/meshes/Gazebo_Base_Body.STL"
               scale="0.001 0.001 0.001" />
       </geometry>
@@ -24,5 +24,5 @@
       <origin xyz="${xd} ${yd} 0" rpy="1.57079 0 0"/>
       <geometry>
-        <mesh filename="package://urdf_tutorial/meshes/Gazebo_Base_Body.STL"
+        <mesh filename="package://urdf_tutorial_r2d2/meshes/Gazebo_Base_Body.STL"
               scale="0.001 0.001 0.001" />
       </geometry>
@@ -32,5 +32,5 @@
     <visual name="arm_1_link_visual">
       <geometry>
-        <mesh filename="package://urdf_tutorial/meshes/Gazebo_Base_arm.STL"
+        <mesh filename="package://urdf_tutorial_r2d2/meshes/Gazebo_Base_arm.STL"
               scale="0.001 0.001 0.001"/>
       </geometry>
@@ -39,5 +39,5 @@
     <collision>
       <geometry>
-        <mesh filename="package://urdf_tutorial/meshes/Gazebo_Base_arm.STL"
+        <mesh filename="package://urdf_tutorial_r2d2/meshes/Gazebo_Base_arm.STL"
               scale="0.001 0.001 0.001"/>
       </geometry>
@@ -48,5 +48,5 @@
     <visual name="arm_2_link_visual">
       <geometry>
-      <mesh filename="package://urdf_tutorial/meshes/Gazebo_Base_arm.STL"
+      <mesh filename="package://urdf_tutorial_r2d2/meshes/Gazebo_Base_arm.STL"
             scale="0.001 0.001 0.001"/>
       </geometry>
@@ -56,5 +56,5 @@
       <origin xyz="0 ${-arm_base} 0"/>
       <geometry>
-        <mesh filename="package://urdf_tutorial/meshes/Gazebo_Base_arm.STL"
+        <mesh filename="package://urdf_tutorial_r2d2/meshes/Gazebo_Base_arm.STL"
               scale="0.001 0.001 0.001"/>
       </geometry>
@@ -64,5 +64,5 @@
     <visual name="arm_3_link_visual">
       <geometry>
-        <mesh filename="package://urdf_tutorial/meshes/Gazebo_Base_arm.STL"
+        <mesh filename="package://urdf_tutorial_r2d2/meshes/Gazebo_Base_arm.STL"
               scale="0.001 0.001 0.001"/>
       </geometry>
@@ -71,5 +71,5 @@
     <collision>
       <geometry>
-        <mesh filename="package://urdf_tutorial/meshes/Gazebo_Base_arm.STL"
+        <mesh filename="package://urdf_tutorial_r2d2/meshes/Gazebo_Base_arm.STL"
               scale="0.001 0.001 0.001"/>
       </geometry>
@@ -80,5 +80,5 @@
     <visual name="arm_4_link_visual">
       <geometry>
-        <mesh filename="package://urdf_tutorial/meshes/Gazebo_Base_arm.STL"
+        <mesh filename="package://urdf_tutorial_r2d2/meshes/Gazebo_Base_arm.STL"
               scale="0.001 0.001 0.001"/>
       </geometry>
@@ -87,5 +87,5 @@
     <collision>
       <geometry>
-        <mesh filename="package://urdf_tutorial/meshes/Gazebo_Base_arm.STL"
+        <mesh filename="package://urdf_tutorial_r2d2/meshes/Gazebo_Base_arm.STL"
               scale="0.001 0.001 0.001"/>
       </geometry>
@@ -124,5 +124,5 @@
     <visual name="prop_1_link_visual">
       <geometry>
-        <mesh filename="package://urdf_tutorial/meshes/1345_prop_ccw.STL"/>
+        <mesh filename="package://urdf_tutorial_r2d2/meshes/1345_prop_ccw.STL"/>
       </geometry>
       <origin  rpy="0 0 0" xyz="-0.03 -0.17 0"/>
@@ -138,5 +138,5 @@
     <visual name="prop_2_link_visual">
       <geometry>
-        <mesh filename="package://urdf_tutorial/meshes/1345_prop_cw.STL"/>
+        <mesh filename="package://urdf_tutorial_r2d2/meshes/1345_prop_cw.STL"/>
       </geometry>
       <origin  rpy="0 0 0" xyz="-0.03 -0.17 0"/>
@@ -152,5 +152,5 @@
     <visual name="prop_3_link_visual">
       <geometry>
-        <mesh filename="package://urdf_tutorial/meshes/1345_prop_ccw.STL"/>
+        <mesh filename="package://urdf_tutorial_r2d2/meshes/1345_prop_ccw.STL"/>
       </geometry>
       <origin  rpy="0 0 0" xyz="-0.03 -0.17 0"/>
@@ -166,5 +166,5 @@
     <visual name="prop_4_link_visual">
       <geometry>
-        <mesh filename="package://urdf_tutorial/meshes/1345_prop_cw.STL"/>
+        <mesh filename="package://urdf_tutorial_r2d2/meshes/1345_prop_cw.STL"/>
       </geometry>
       <origin  rpy="0 0 0" xyz="-0.03 -0.17 0"/>
