Commit message: renaming rospackage

File: ros_pack/projet_robo_redev/urdf/4arms.urdf (robot description, URDF)
Before this commit: robot 4Armdrone, 9 links, 8 joints
Links:
- link arm_1: geometry collision mesh filename=package://projet_robo_redev/meshes/Gazebo_Base_arm.stl scale=0.001 0.001 0.001; visual mesh filename=package://projet_robo_redev/meshes/Gazebo_Base_arm.stl scale=0.001 0.001 0.001
- link arm_2: geometry collision mesh filename=package://projet_robo_redev/meshes/Gazebo_Base_arm.stl scale=0.001 0.001 0.001; visual mesh filename=package://projet_robo_redev/meshes/Gazebo_Base_arm.stl scale=0.001 0.001 0.001
- link arm_3: geometry collision mesh filename=package://projet_robo_redev/meshes/Gazebo_Base_arm.stl scale=0.001 0.001 0.001; visual mesh filename=package://projet_robo_redev/meshes/Gazebo_Base_arm.stl scale=0.001 0.001 0.001
- link arm_4: geometry collision mesh filename=package://projet_robo_redev/meshes/Gazebo_Base_arm.stl scale=0.001 0.001 0.001; visual mesh filename=package://projet_robo_redev/meshes/Gazebo_Base_arm.stl scale=0.001 0.001 0.001
- link drone: geometry collision mesh filename=package://projet_robo_redev/meshes/Gazebo_Base_Body.stl scale=0.001 0.001 0.001; visual mesh filename=package://projet_robo_redev/meshes/Gazebo_Base_Body.stl scale=0.001 0.001 0.001
- link prop_1: geometry visual mesh filename=package://projet_robo_redev/meshes/1345_prop_ccw.stl
- link prop_2: geometry visual mesh filename=package://projet_robo_redev/meshes/1345_prop_cw.stl
- link prop_3: geometry visual mesh filename=package://projet_robo_redev/meshes/1345_prop_ccw.stl
- link prop_4: geometry visual mesh filename=package://projet_robo_redev/meshes/1345_prop_cw.stl

File: ros_pack/projet_robo_redev/urdf/4arms.urdf.xacro (robot description, xacro)
@@ -1,12 +1,20 @@
 <?xml version="1.0"?>
-<robot name="4ArmDrone">
+<robot name="4Armdrone"  xmlns:xacro="http://www.ros.org/wiki/xacro">
   <material name="blue">
     <color rgba="0 0 0.8 1"/>
   </material>
-  <link name="base_link">
-    <visual name="base_link_visual">
-      <origin xyz="0 0 0" rpy="1.57079 0 0"/>
+<xacro:property name='sktX' value="0.19674"/>
+<xacro:property name='sktY' value="0.09329"/>
+<xacro:property name="xd"   value="${-sktX/2}"/>
+<xacro:property name="yd"   value="${sktY/2}"/>
+<xacro:property name="arm_junction" value="0.0293"/>
+<xacro:property name="arm_base" value="0.035"/>
+<xacro:property name="arm_ang" value="0.5788"/>
+<xacro:property name="arm_len" value="0.155"/>
+  <link name="drone">
+    <visual name="drone_visual">
+      <origin xyz="${xd} ${yd} 0" rpy="1.57079 0 0"/>
       <geometry>
-        <mesh filename="package://urdf_tutorial/meshes/Gazebo_Base_Body.stl"
+        <mesh filename="package://projet_robo_redev/meshes/Gazebo_Base_Body.stl"
               scale="0.001 0.001 0.001" />
       </geometry>
@@ -14,7 +22,7 @@
     </visual>
     <collision>
-      <origin xyz="0 0 0" rpy="1.57079 0 0"/>
+      <origin xyz="${xd} ${yd} 0" rpy="1.57079 0 0"/>
       <geometry>
-        <mesh filename="package://urdf_tutorial/meshes/Gazebo_Base_Body.stl"
+        <mesh filename="package://projet_robo_redev/meshes/Gazebo_Base_Body.stl"
               scale="0.001 0.001 0.001" />
       </geometry>
@@ -24,13 +32,15 @@
     <visual name="arm_1_link_visual">
       <geometry>
-        <mesh filename="package://urdf_tutorial/meshes/Gazebo_Base_arm.stl"
+        <mesh filename="package://projet_robo_redev/meshes/Gazebo_Base_arm.stl"
               scale="0.001 0.001 0.001"/>
       </geometry>
+      <origin xyz="0 ${0} 0"/>
     </visual>
     <collision>
       <geometry>
-        <mesh filename="package://urdf_tutorial/meshes/Gazebo_Base_arm.stl"
+        <mesh filename="package://projet_robo_redev/meshes/Gazebo_Base_arm.stl"
               scale="0.001 0.001 0.001"/>
       </geometry>
+      <origin xyz="0 ${0} 0"/>
     </collision>
   </link>
@@ -38,13 +48,13 @@
     <visual name="arm_2_link_visual">
       <geometry>
-      <mesh filename="package://urdf_tutorial/meshes/Gazebo_Base_arm.stl"
+      <mesh filename="package://projet_robo_redev/meshes/Gazebo_Base_arm.stl"
             scale="0.001 0.001 0.001"/>
       </geometry>
-      <origin xyz="0 -0.035 0"/>
+      <origin xyz="0 ${-arm_base} 0"/>
     </visual>
     <collision>
-      <origin xyz="0 -0.035 0"/>
+      <origin xyz="0 ${-arm_base} 0"/>
       <geometry>
-        <mesh filename="package://urdf_tutorial/meshes/Gazebo_Base_arm.stl"
+        <mesh filename="package://projet_robo_redev/meshes/Gazebo_Base_arm.stl"
               scale="0.001 0.001 0.001"/>
       </geometry>
@@ -54,13 +64,15 @@
     <visual name="arm_3_link_visual">
       <geometry>
-        <mesh filename="package://urdf_tutorial/meshes/Gazebo_Base_arm.stl"
+        <mesh filename="package://projet_robo_redev/meshes/Gazebo_Base_arm.stl"
               scale="0.001 0.001 0.001"/>
       </geometry>
+      <origin xyz="0 ${0} 0"/>
     </visual>
     <collision>
       <geometry>
-        <mesh filename="package://urdf_tutorial/meshes/Gazebo_Base_arm.stl"
+        <mesh filename="package://projet_robo_redev/meshes/Gazebo_Base_arm.stl"
               scale="0.001 0.001 0.001"/>
       </geometry>
+      <origin xyz="0 ${0} 0"/>
     </collision>
   </link>
@@ -68,42 +80,42 @@
     <visual name="arm_4_link_visual">
       <geometry>
-        <mesh filename="package://urdf_tutorial/meshes/Gazebo_Base_arm.stl"
+        <mesh filename="package://projet_robo_redev/meshes/Gazebo_Base_arm.stl"
               scale="0.001 0.001 0.001"/>
       </geometry>
-      <origin xyz="0 -0.035 0"/>
+      <origin xyz="0 ${-arm_base} 0"/>
     </visual>
     <collision>
       <geometry>
-        <mesh filename="package://urdf_tutorial/meshes/Gazebo_Base_arm.stl"
+        <mesh filename="package://projet_robo_redev/meshes/Gazebo_Base_arm.stl"
               scale="0.001 0.001 0.001"/>
       </geometry>
-      <origin xyz="0 -0.035 0"/>
+      <origin xyz="0 ${-arm_base} 0"/>
     </collision>
   </link>
   <joint name="base_to_arm_1" type="revolute">
-    <parent link="base_link"/>
+    <parent link="drone"/>
     <child link="arm_1"/>
-    <origin  rpy="0 0 2.15" xyz="0.029 0 0"/>
+    <origin  rpy="0 0 ${pi/2+arm_ang}" xyz="${xd+arm_junction} ${yd} 0"/>
     <axis xyz="0.0 1.0 0.0"/>
     <limit effort="1000.0" lower="0.0" upper="1.74" velocity="1000.0"/>
   </joint>
   <joint name="base_to_arm_2" type="revolute">
-    <parent link="base_link"/>
+    <parent link="drone"/>
     <child link="arm_2"/>
-    <origin  rpy="0 0 -2.15" xyz="0.029 -0.093 0"/>
+    <origin  rpy="0 0 -${pi/2+arm_ang}" xyz="${xd+arm_junction} ${-yd} 0"/>
     <axis xyz="0.0 1.0 0.0"/>
     <limit effort="1000.0" lower="0.0" upper="1.74" velocity="1000.0"/>
   </joint>
   <joint name="base_to_arm_3" type="revolute">
-    <parent link="base_link"/>
+    <parent link="drone"/>
     <child link="arm_3"/>
-    <origin  rpy="0 0 -1" xyz="0.165 -0.093 0"/>
+    <origin  rpy="0 0 -${pi/2-arm_ang}" xyz="${-xd-arm_junction} ${-yd} 0"/>
     <axis xyz="0.0 1.0 0.0"/>
     <limit effort="1000.0" lower="0.0" upper="1.74" velocity="1000.0"/>
   </joint>
   <joint name="base_to_arm_4" type="revolute">
-    <parent link="base_link"/>
+    <parent link="drone"/>
     <child link="arm_4"/>
-    <origin  rpy="0 0 1" xyz="0.165 0.0 0"/>
+    <origin  rpy="0 0 ${pi/2-arm_ang}" xyz="${-xd-arm_junction} ${yd} 0"/>
     <axis xyz="0.0 1.0 0.0"/>
     <limit effort="1000.0" lower="0.0" upper="1.74" velocity="1000.0"/>
@@ -112,5 +124,5 @@
     <visual name="prop_1_link_visual">
       <geometry>
-        <mesh filename="package://urdf_tutorial/meshes/1345_prop_ccw.stl"/>
+        <mesh filename="package://projet_robo_redev/meshes/1345_prop_ccw.stl"/>
       </geometry>
       <origin  rpy="0 0 0" xyz="-0.03 -0.17 0"/>
@@ -120,5 +132,5 @@
     <parent link="arm_1"/>
     <child link="prop_1"/>
-    <origin  rpy="0 0 0" xyz="0.17 0.02 0.03"/>
+    <origin  rpy="0 0 0" xyz="${arm_len} ${arm_base/2} ${0}"/>
     <axis xyz="0.0 0.0 1"/>
   </joint>
@@ -126,5 +138,5 @@
     <visual name="prop_2_link_visual">
       <geometry>
-        <mesh filename="package://urdf_tutorial/meshes/1345_prop_cw.stl"/>
+        <mesh filename="package://projet_robo_redev/meshes/1345_prop_cw.stl"/>
       </geometry>
       <origin  rpy="0 0 0" xyz="-0.03 -0.17 0"/>
@@ -134,11 +146,11 @@
     <parent link="arm_2"/>
     <child link="prop_2"/>
-    <origin  rpy="0 0 0" xyz="0.17 -0.02 0.03"/>
-    <axis xyz="0.0 0.0 -1"/>
+    <origin  rpy="0 0 0" xyz="${arm_len} ${-arm_base/2} ${0}"/>
+    <axis xyz="0.0 0.0 1"/>
   </joint>
   <link name="prop_3">
     <visual name="prop_3_link_visual">
       <geometry>
-        <mesh filename="package://urdf_tutorial/meshes/1345_prop_ccw.stl"/>
+        <mesh filename="package://projet_robo_redev/meshes/1345_prop_ccw.stl"/>
       </geometry>
       <origin  rpy="0 0 0" xyz="-0.03 -0.17 0"/>
@@ -148,5 +160,5 @@
     <parent link="arm_3"/>
     <child link="prop_3"/>
-    <origin  rpy="0 0 0" xyz="0.17 0.02 0.03"/>
+    <origin  rpy="0 0 0" xyz="${arm_len} ${arm_base/2} ${0}"/>
     <axis xyz="0.0 0.0 1"/>
   </joint>
@@ -154,5 +166,5 @@
     <visual name="prop_4_link_visual">
       <geometry>
-        <mesh filename="package://urdf_tutorial/meshes/1345_prop_cw.stl"/>
+        <mesh filename="package://projet_robo_redev/meshes/1345_prop_cw.stl"/>
       </geometry>
       <origin  rpy="0 0 0" xyz="-0.03 -0.17 0"/>
@@ -162,6 +174,6 @@
     <parent link="arm_4"/>
     <child link="prop_4"/>
-    <origin  rpy="0 0 0" xyz="0.17 -0.02 0.03"/>
-    <axis xyz="0.0 0.0 -1"/>
+    <origin  rpy="0 0 0" xyz="${arm_len} ${-arm_base/2} ${0}"/>
+    <axis xyz="0.0 0.0 1"/>
   </joint>
 </robot>
